File: processor.kicad_sch (KiCad schematic)
At the start: 28 parts, among them J6 Conn_Coaxial, SW1 SW-434153017835‎, SW2 SW-434153017835‎, U10 SKY65723-81, U12 nRF9151-LAXX, U3 1042240820, U4 W25Q128JVPIQ, U6 SIM-ST-MFF2

Commit message: Updating parts:
1. Button change
2. USB change
Parts:
- SW1, SW2: footprint Circuit Dojo:WOLFF-DEN_SW-EVP-AA402W -> Button_Switch_SMD:SW_SPST_B3U-1000P
Changed lines of the file:
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@@
 			)
 		)
-		(property "Footprint" "Circuit Dojo:WOLFF-DEN_SW-EVP-AA402W"
+		(property "Footprint" "Button_Switch_SMD:SW_SPST_B3U-1000P"
 			(at 100.33 208.28 0)
 			(effects
@@
 			)
 		)
-		(property "Footprint" "Circuit Dojo:WOLFF-DEN_SW-EVP-AA402W"
+		(property "Footprint" "Button_Switch_SMD:SW_SPST_B3U-1000P"
 			(at 64.77 250.19 0)
 			(effects
